Commit message: Adding ros2 control support

File: orion_simulation/description/urdf/diff_wheels.urdf.xacro (robot description, xacro)
@@ -19,4 +19,7 @@
     </xacro:inertial_cylinder>
     </link>
+    <gazebo reference="chassis">
+        <material>Gazebo/Blue</material>
+    </gazebo>
 </xacro:macro>
 </robot>

File: orion_simulation/description/urdf/robot.urdf.xacro (robot description, xacro)
@@ -4,4 +4,5 @@
 <xacro:include filename="$(find orion_simulation)/description/urdf/diff_wheels.urdf.xacro"/>
 <xacro:include filename="$(find orion_simulation)/description/urdf/inertial_macros.xacro" />
+<xacro:include filename="$(find orion_simulation)/description/urdf/gazebo_control.xacro" />
 <!-- Robot Base -->
 <link name="base_link"> </link>
@@ -11,4 +12,5 @@
     <origin xyz="-0.1 0 0"/>
 </joint>
+<!-- Base Chassis -->
 <link name="chassis">
     <visual>
@@ -29,7 +31,11 @@
     </xacro:inertial_box>
 </link>
-<!-- LEFT WHEEL -->
+<gazebo reference="chassis">
+    <material>Gazebo/White</material>
+</gazebo>
+<!-- Diff Wheels -->
 <xacro:wheel prefix="left" reflect="1" />
 <xacro:wheel prefix="right" reflect="-1" />
+<!-- Caster Wheels -->
 <joint name="caster_wheel_joint" type="fixed">
     <parent link="chassis"/>
@@ -48,3 +54,8 @@
     </xacro:inertial_sphere>
 </link>
+<gazebo reference="chassis">
+    <material>Gazebo/Black</material>
+    <mu1 value="0.001"/>
+    <mu2 value="0.001"/>
+</gazebo>
 </robot>

Commit message: Teleop twist controlling robot through Ros2 Control

File: orion_simulation/description/urdf/diff_wheels.urdf.xacro (robot description, xacro)
@@ -15,11 +15,13 @@
         <material name="blue"/>
     </visual>
+     <collision>
+        <geometry>
+            <sphere radius="${diff_wheel_radius}"/>
+        </geometry>
+    </collision>
     <xacro:inertial_cylinder mass="0.1" length="0.05" radius="0.05">
         <origin xyz="0 0 0" rpy="0 0 0"/>
     </xacro:inertial_cylinder>
     </link>
-    <gazebo reference="chassis">
-        <material>Gazebo/Blue</material>
-    </gazebo>
 </xacro:macro>
 </robot>

File: orion_simulation/description/urdf/robot.urdf.xacro (robot description, xacro)
@@ -31,7 +31,4 @@
     </xacro:inertial_box>
 </link>
-<gazebo reference="chassis">
-    <material>Gazebo/White</material>
-</gazebo>
 <!-- Diff Wheels -->
 <xacro:wheel prefix="left" reflect="1" />
@@ -43,19 +40,24 @@
     <origin xyz="0.24 0 0" rpy="0 0 0"/>
 </joint>
-<link name="caster_wheel">
-    <visual>
-        <geometry>
-            <sphere radius="0.05" />
-        </geometry>
-        <material name="black"/>
-    </visual>
-    <xacro:inertial_sphere mass="0.1" radius="0.05">
-      <origin xyz="0 0 0" rpy="0 0 0"/>
-    </xacro:inertial_sphere>
-</link>
-<gazebo reference="chassis">
-    <material>Gazebo/Black</material>
-    <mu1 value="0.001"/>
-    <mu2 value="0.001"/>
-</gazebo>
+ <link name="caster_wheel">
+        <visual>
+            <geometry>
+                <sphere radius="${caster_wheel_radius}"/>
+            </geometry>
+            <material name="white"/>
+        </visual>
+        <collision>
+            <geometry>
+                <sphere radius="${caster_wheel_radius}"/>
+            </geometry>
+        </collision>
+        <xacro:inertial_sphere mass="10" radius="${caster_wheel_radius}">
+            <origin xyz="0 0 0" rpy="0 0 0"/>
+        </xacro:inertial_sphere>
+    </link>
+    <gazebo reference="caster_wheel">
+        <material>Gazebo/Blue</material>
+        <mu1 value="0.01"/>
+        <mu2 value="0.01"/>
+    </gazebo>
 </robot>

File: orion_simulation/description/urdf/robot_properties.urdf.xacro (robot description, xacro)
@@ -8,5 +8,5 @@
   <xacro:property name="diff_wheel_width" value="0.02" />
   <xacro:property name="diff_wheel_y" value="0.175" />
-  <xacro:property name="caster_wheel_radius" value="0.02" />
+  <xacro:property name="caster_wheel_radius" value="0.05" />
   <material name="white">
     <color rgba="1 1 1 1"/>

File: orion_simulation/description/urdf/ros2_control.xacro (robot description, xacro)
@@ -6,15 +6,23 @@
         </hardware>
         <joint name="left_wheel_joint">
-            <command_interface name="velocity"/>
-            <state_interface name="velocity"/>
+            <command_interface name="velocity">
+                <param name="min">-10</param>
+                <param name="max">10</param>
+            </command_interface>
+            <state_interface name="position" />
+            <state_interface name="velocity" />
         </joint>
         <joint name="right_wheel_joint">
-            <command_interface name="velocity"/>
-            <state_interface name="velocity"/>
+            <command_interface name="velocity">
+                <param name="min">-10</param>
+                <param name="max">10</param>
+            </command_interface>
+            <state_interface name="velocity" />
+            <state_interface name="position" />
         </joint>
     </ros2_control>
     <gazebo>
-        <plugin filename="gz_ros2_control-system" name="gz_ros2_control::GazeboSimROS2ControlPlugin">
-            <parameters>$(find orion_simulation)/config/controller.yaml</parameters>
+        <plugin name="gz_ros2_control::GazeboSimROS2ControlPlugin" filename="libgz_ros2_control-system.so">
+            <parameters>$(find orion_simulation)/config/diff_drive_controller.yaml</parameters>
         </plugin>
     </gazebo>
