Commit message: Added lidar to simulation, adding new urdf and updating gz_bridge.yaml

File: orion_description/urdf/robot.urdf.xacro (robot description, xacro)
@@ -4,5 +4,6 @@
 <xacro:include filename="$(find orion_description)/urdf/diff_wheels.urdf.xacro"/>
 <xacro:include filename="$(find orion_description)/urdf/inertial_macros.xacro" />
-<!-- <xacro:include filename="$(find orion_description)/urdf/ros2_control.xacro" /> -->
+<xacro:include filename="$(find orion_description)/urdf/lidar.xacro" />
+<xacro:include filename="$(find orion_description)/urdf/ros2_control.xacro" />
 <!-- Robot Base -->
 <link name="base_link"> </link>

File: orion_description/urdf/robot_properties.urdf.xacro (robot description, xacro)
@@ -9,4 +9,6 @@
   <xacro:property name="diff_wheel_y" value="0.175" />
   <xacro:property name="caster_wheel_radius" value="0.05" />
+  <xacro:property name="lidar_radius" value="0.05" />
+  <xacro:property name="lidar_length" value="0.04" />
   <material name="white">
     <color rgba="1 1 1 1"/>

Commit message: Added a camera to work in IGN simulation

File: orion_description/urdf/robot.urdf.xacro (robot description, xacro)
@@ -5,4 +5,5 @@
 <xacro:include filename="$(find orion_description)/urdf/inertial_macros.xacro" />
 <xacro:include filename="$(find orion_description)/urdf/lidar.xacro" />
+<xacro:include filename="$(find orion_description)/urdf/camera.xacro" />
 <xacro:include filename="$(find orion_description)/urdf/ros2_control.xacro" />
 <!-- Robot Base -->

File: orion_description/urdf/robot_properties.urdf.xacro (robot description, xacro)
@@ -11,4 +11,7 @@
   <xacro:property name="lidar_radius" value="0.05" />
   <xacro:property name="lidar_length" value="0.04" />
+  <xacro:property name="camera_width" value="0.02" />
+  <xacro:property name="camera_height" value="0.075" />
+  <xacro:property name="camera_length" value="0.075" />
   <material name="white">
     <color rgba="1 1 1 1"/>
